Commit message: -

File: src/bigspot_description/urdf/bigspot.xacro (robot description, xacro)
@@ -297,5 +297,5 @@
   <child link="RLF_1"/>
   <axis xyz="0.013454 0.999909 0.001153"/>
-  <limit upper="1.22173" lower="-1.22173" effort="3.5" velocity="3"/>
+  <limit upper="1.22173" lower="-1.22173" effort="3.0" velocity="3"/>
 </joint>
 <joint name="RRF_Joint" type="revolute">
@@ -304,5 +304,5 @@
   <child link="RRF_1"/>
   <axis xyz="0.001225 -0.99999 0.004366"/>
-  <limit upper="1.22173" lower="-1.22173" effort="3.5" velocity="3"/>
+  <limit upper="1.22173" lower="-1.22173" effort="3.0" velocity="3"/>
 </joint>
 <joint name="FRF_Joint" type="revolute">
@@ -311,5 +311,5 @@
   <child link="FRF_1"/>
   <axis xyz="-0.002804 -0.999995 0.001625"/>
-  <limit upper="1.22173" lower="-1.22173" effort="3.5" velocity="3"/>
+  <limit upper="1.22173" lower="-1.22173" effort="3.0" velocity="3"/>
 </joint>
 <joint name="FLF_Joint" type="revolute">
@@ -318,5 +318,5 @@
   <child link="FLF_1"/>
   <axis xyz="0.002803 0.999992 -0.002813"/>
-  <limit upper="1.22173" lower="-1.22173" effort="3.5" velocity="3"/>
+  <limit upper="1.22173" lower="-1.22173" effort="3.0" velocity="3"/>
 </joint>
 <joint name="FRL_Joint" type="revolute">
@@ -325,5 +325,5 @@
   <child link="FRL_1"/>
   <axis xyz="0.002804 0.999995 -0.001625"/>
-  <limit upper="1.22173" lower="-1.22173" effort="3.5" velocity="3"/>
+  <limit upper="1.22173" lower="-1.22173" effort="3.0" velocity="3"/>
 </joint>
 <joint name="FLL_Joint" type="revolute">
@@ -332,5 +332,5 @@
   <child link="FLL_1"/>
   <axis xyz="-0.002803 -0.999992 0.002813"/>
-  <limit upper="1.22173" lower="-1.22173" effort="3.5" velocity="3"/>
+  <limit upper="1.22173" lower="-1.22173" effort="3.0" velocity="3"/>
 </joint>
 <joint name="RLL_Joint" type="revolute">
@@ -339,5 +339,5 @@
   <child link="RLL_1"/>
   <axis xyz="-0.001768 -0.999997 0.001824"/>
-  <limit upper="1.22173" lower="-1.22173" effort="3.5" velocity="3"/>
+  <limit upper="1.22173" lower="-1.22173" effort="3.0" velocity="3"/>
 </joint>
 <joint name="RRL_Joint" type="revolute">
@@ -346,5 +346,161 @@
   <child link="RRL_1"/>
   <axis xyz="0.001768 0.999998 -0.000636"/>
-  <limit upper="1.22173" lower="-1.22173" effort="3.5" velocity="3"/>
-</joint>
+  <limit upper="1.22173" lower="-1.22173" effort="3.0" velocity="3"/>
+</joint>
+<!-- RR4 -->
+<link name="RR4">
+  <inertial>
+    <origin
+      xyz="0.00 0 0"
+      rpy="0 0 0" />
+   <mass
+      value="0.0391" />
+    <inertia
+      ixx="3.7713E-012"
+      ixy="0"
+      ixz="0"
+      iyy="3.5422E-12"
+      iyz="0"
+      izz="5.443E-012" />
+  </inertial>
+  <collision>
+    <origin
+      xyz="0 0 0"
+      rpy="0 0 0" />
+    <geometry>
+      <sphere radius="0.0072"/>
+    </geometry>
+  </collision>
+</link>
+<!-- RR4 -->
+<link name="RL4">
+  <inertial>
+    <origin
+      xyz="0.00 0 0"
+      rpy="0 0 0" />
+   <mass
+      value="0.0391" />
+    <inertia
+      ixx="3.7713E-012"
+      ixy="0"
+      ixz="0"
+      iyy="3.5422E-12"
+      iyz="0"
+      izz="5.443E-012" />
+  </inertial>
+  <collision>
+    <origin
+      xyz="0 0 0"
+      rpy="0 0 0" />
+    <geometry>
+      <sphere radius="0.0072"/>
+    </geometry>
+  </collision>
+</link>
+<!-- RR4 -->
+<link name="FR4">
+  <inertial>
+    <origin
+      xyz="0.00 0 0"
+      rpy="0 0 0" />
+   <mass
+      value="0.0391" />
+    <inertia
+      ixx="3.7713E-012"
+      ixy="0"
+      ixz="0"
+      iyy="3.5422E-12"
+      iyz="0"
+      izz="5.443E-012" />
+  </inertial>
+  <collision>
+    <origin
+      xyz="0 0 0"
+      rpy="0 0 0" />
+    <geometry>
+      <sphere radius="0.0072"/>
+    </geometry>
+  </collision>
+</link>
+<!-- RR4 -->
+<link name="FL4">
+  <inertial>
+    <origin
+      xyz="0.00 0 0"
+      rpy="0 0 0" />
+   <mass
+      value="0.0391" />
+    <inertia
+      ixx="3.7713E-012"
+      ixy="0"
+      ixz="0"
+      iyy="3.5422E-12"
+      iyz="0"
+      izz="5.443E-012" />
+  </inertial>
+  <collision>
+    <origin
+      xyz="0 0 0"
+      rpy="0 0 0" />
+    <geometry>
+      <sphere radius="0.0072"/>
+    </geometry>
+  </collision>
+</link>
+<joint name="RR4_Joint" type="fixed">
+  <origin xyz="0.094333 0 0" rpy="0 0 0" />
+  <parent link="RRF_1" />
+  <child link="RR4" />
+  <axis xyz="0 0 0" />
+</joint>
+<!-- RR4 friction -->
+<gazebo reference="RR4">
+  <mu1>1.0</mu1>
+  <mu2>1.0</mu2>
+  <minDepth>0.0002</minDepth>
+  <kp  value="1000000.0"/>
+  <kd  value="100.0"/>
+</gazebo>
+<joint name="RL4_Joint" type="fixed">
+  <origin xyz="0.094333 0 0" rpy="0 0 0" />
+  <parent link="RLF_1" />
+  <child link="RL4" />
+  <axis xyz="0 0 0" />
+</joint>
+<!-- RR4 friction -->
+<gazebo reference="RL4">
+  <mu1>1.0</mu1>
+  <mu2>1.0</mu2>
+  <minDepth>0.0002</minDepth>
+  <kp  value="1000000.0"/>
+  <kd  value="100.0"/>
+</gazebo>
+<joint name="FR4_Joint" type="fixed">
+  <origin xyz="0.094333 0 0" rpy="0 0 0" />
+  <parent link="FRF_1" />
+  <child link="FR4" />
+  <axis xyz="0 0 0" />
+</joint>
+<!-- RR4 friction -->
+<gazebo reference="FR4">
+  <mu1>1.0</mu1>
+  <mu2>1.0</mu2>
+  <minDepth>0.0002</minDepth>
+  <kp  value="1000000.0"/>
+  <kd  value="100.0"/>
+</gazebo>
+<joint name="FL4_Joint" type="fixed">
+  <origin xyz="0.094333 0 0" rpy="0 0 0" />
+  <parent link="FLF_1" />
+  <child link="FL4" />
+  <axis xyz="0 0 0" />
+</joint>
+<!-- RR4 friction -->
+<gazebo reference="FL4">
+  <mu1>1.0</mu1>
+  <mu2>1.0</mu2>
+  <minDepth>0.0002</minDepth>
+  <kp  value="1000000.0"/>
+  <kd  value="100.0"/>
+</gazebo>
 </robot>

Commit message: -

File: src/bigspot_description/urdf/bigspot.xacro (robot description, xacro)
@@ -6,7 +6,7 @@
 <link name="base_link">
   <inertial>
-    <origin xyz="0.0311133655846206 -0.0004882003232346135 0.33321366100631183" rpy="0 0 0"/>
-    <mass value="1.2008096267597053"/>
-    <inertia ixx="0.003822" iyy="0.017546" izz="0.01806" ixy="-0.000113" iyz="-2.3e-05" ixz="0.000214"/>
+    <origin xyz="-0.005924455452065034 -0.00013954843544972099 0.33234964114268223" rpy="0 0 0"/>
+    <mass value="1.2002032804157028"/>
+    <inertia ixx="0.003833" iyy="0.01767" izz="0.018171" ixy="-0.000152" iyz="-3.3e-05" ixz="-8e-05"/>
   </inertial>
   <visual>
@@ -24,12 +24,72 @@
   </collision>
 </link>
+<link name="FRS_1">
+  <inertial>
+    <origin xyz="-0.03262402906297844 -0.008891213440249235 -0.01859885653575638" rpy="0 0 0"/>
+    <mass value="0.2179660102657959"/>
+    <inertia ixx="0.00014" iyy="0.000135" izz="9.7e-05" ixy="2e-06" iyz="-0.0" ixz="-3e-06"/>
+  </inertial>
+  <visual>
+    <origin xyz="-0.152485 0.048774 -0.341762" rpy="0 0 0"/>
+    <geometry>
+      <mesh filename="package://bigspot_description/meshes/FRS_1.stl" scale="0.001 0.001 0.001"/>
+    </geometry>
+    <material name="silver"/>
+  </visual>
+  <collision>
+    <origin xyz="-0.152485 0.048774 -0.341762" rpy="0 0 0"/>
+    <geometry>
+      <mesh filename="package://bigspot_description/meshes/FRS_1.stl" scale="0.001 0.001 0.001"/>
+    </geometry>
+  </collision>
+</link>
+<link name="FRL_1">
+  <inertial>
+    <origin xyz="0.0038775817781630667 -0.033503810432042994 -0.051270367340440826" rpy="0 0 0"/>
+    <mass value="0.2533070021724165"/>
+    <inertia ixx="0.000608" iyy="0.000566" izz="0.000103" ixy="4e-06" iyz="-3.8e-05" ixz="4e-05"/>
+  </inertial>
+  <visual>
+    <origin xyz="-0.121434 0.09266 -0.322919" rpy="0 0 0"/>
+    <geometry>
+      <mesh filename="package://bigspot_description/meshes/FRL_1.stl" scale="0.001 0.001 0.001"/>
+    </geometry>
+    <material name="silver"/>
+  </visual>
+  <collision>
+    <origin xyz="-0.121434 0.09266 -0.322919" rpy="0 0 0"/>
+    <geometry>
+      <mesh filename="package://bigspot_description/meshes/FRL_1.stl" scale="0.001 0.001 0.001"/>
+    </geometry>
+  </collision>
+</link>
+<link name="FRF_1">
+  <inertial>
+    <origin xyz="-0.001869412585041974 -0.03622957158869643 -0.04650897056843453" rpy="0 0 0"/>
+    <mass value="0.25008271350190114"/>
+    <inertia ixx="0.000701" iyy="0.000678" izz="7e-05" ixy="0.0" iyz="2e-06" ixz="9e-06"/>
+  </inertial>
+  <visual>
+    <origin xyz="-0.145661 0.096431 -0.182302" rpy="0 0 0"/>
+    <geometry>
+      <mesh filename="package://bigspot_description/meshes/FRF_1.stl" scale="0.001 0.001 0.001"/>
+    </geometry>
+    <material name="silver"/>
+  </visual>
+  <collision>
+    <origin xyz="-0.145661 0.096431 -0.182302" rpy="0 0 0"/>
+    <geometry>
+      <mesh filename="package://bigspot_description/meshes/FRF_1.stl" scale="0.001 0.001 0.001"/>
+    </geometry>
+  </collision>
+</link>
 <link name="FLS_1">
   <inertial>
-    <origin xyz="0.031987412635341245 -0.009034675998087056 -0.018895160159360047" rpy="0 0 0"/>
-    <mass value="0.21643936164319344"/>
-    <inertia ixx="0.000138" iyy="0.000133" izz="9.5e-05" ixy="-2e-06" iyz="-0.0" ixz="4e-06"/>
-  </inertial>
-  <visual>
-    <origin xyz="0.132847 0.048403 -0.342309" rpy="0 0 0"/>
+    <origin xyz="-0.032502651385048306 0.008982081400929244 -0.01876110043924245" rpy="0 0 0"/>
+    <mass value="0.2168042558568771"/>
+    <inertia ixx="0.000138" iyy="0.000133" izz="9.6e-05" ixy="-1e-06" iyz="0.0" ixz="-4e-06"/>
+  </inertial>
+  <visual>
+    <origin xyz="-0.152487 -0.049214 -0.341737" rpy="0 0 0"/>
     <geometry>
       <mesh filename="package://bigspot_description/meshes/FLS_1.stl" scale="0.001 0.001 0.001"/>
@@ -38,5 +98,5 @@
   </visual>
   <collision>
-    <origin xyz="0.132847 0.048403 -0.342309" rpy="0 0 0"/>
+    <origin xyz="-0.152487 -0.049214 -0.341737" rpy="0 0 0"/>
     <geometry>
       <mesh filename="package://bigspot_description/meshes/FLS_1.stl" scale="0.001 0.001 0.001"/>
@@ -44,21 +104,41 @@
   </collision>
 </link>
-<link name="RFS_1">
-  <inertial>
-    <origin xyz="0.03264566963287516 0.00874581726337579 -0.018745684169703347" rpy="0 0 0"/>
-    <mass value="0.21757543557281156"/>
-    <inertia ixx="0.000139" iyy="0.000135" izz="9.6e-05" ixy="2e-06" iyz="0.0" ixz="3e-06"/>
-  </inertial>
-  <visual>
-    <origin xyz="0.132572 -0.049597 -0.342338" rpy="0 0 0"/>
-    <geometry>
-      <mesh filename="package://bigspot_description/meshes/RFS_1.stl" scale="0.001 0.001 0.001"/>
-    </geometry>
-    <material name="silver"/>
-  </visual>
-  <collision>
-    <origin xyz="0.132572 -0.049597 -0.342338" rpy="0 0 0"/>
-    <geometry>
-      <mesh filename="package://bigspot_description/meshes/RFS_1.stl" scale="0.001 0.001 0.001"/>
+<link name="FLL_1">
+  <inertial>
+    <origin xyz="0.0038795073898601623 0.033676971098066916 -0.0511565901145839" rpy="0 0 0"/>
+    <mass value="0.2533070083934759"/>
+    <inertia ixx="0.000608" iyy="0.000566" izz="0.000103" ixy="-4e-06" iyz="4e-05" ixz="4e-05"/>
+  </inertial>
+  <visual>
+    <origin xyz="-0.12144 -0.092922 -0.323041" rpy="0 0 0"/>
+    <geometry>
+      <mesh filename="package://bigspot_description/meshes/FLL_1.stl" scale="0.001 0.001 0.001"/>
+    </geometry>
+    <material name="silver"/>
+  </visual>
+  <collision>
+    <origin xyz="-0.12144 -0.092922 -0.323041" rpy="0 0 0"/>
+    <geometry>
+      <mesh filename="package://bigspot_description/meshes/FLL_1.stl" scale="0.001 0.001 0.001"/>
+    </geometry>
+  </collision>
+</link>
+<link name="FLF_1">
+  <inertial>
+    <origin xyz="-0.001867050204165388 0.036386780395052415 -0.04638544366195871" rpy="0 0 0"/>
+    <mass value="0.25008282200400833"/>
+    <inertia ixx="0.000701" iyy="0.000678" izz="7e-05" ixy="-0.0" iyz="-0.0" ixz="9e-06"/>
+  </inertial>
+  <visual>
+    <origin xyz="-0.145667 -0.097168 -0.182437" rpy="0 0 0"/>
+    <geometry>
+      <mesh filename="package://bigspot_description/meshes/FLF_1.stl" scale="0.001 0.001 0.001"/>
+    </geometry>
+    <material name="silver"/>
+  </visual>
+  <collision>
+    <origin xyz="-0.145667 -0.097168 -0.182437" rpy="0 0 0"/>
+    <geometry>
+      <mesh filename="package://bigspot_description/meshes/FLF_1.stl" scale="0.001 0.001 0.001"/>
     </geometry>
   </collision>
@@ -66,10 +146,10 @@
 <link name="RRS_1">
   <inertial>
-    <origin xyz="-0.03261704424738682 0.008913094723832414 -0.01871850172783035" rpy="0 0 0"/>
-    <mass value="0.217579149442337"/>
-    <inertia ixx="0.000139" iyy="0.000135" izz="9.6e-05" ixy="-2e-06" iyz="0.0" ixz="-3e-06"/>
-  </inertial>
-  <visual>
-    <origin xyz="-0.184517 -0.048857 -0.342398" rpy="0 0 0"/>
+    <origin xyz="0.0327134074105363 -0.008946282789402397 -0.01858381030389067" rpy="0 0 0"/>
+    <mass value="0.2178784733170752"/>
+    <inertia ixx="0.000139" iyy="0.000135" izz="9.7e-05" ixy="-2e-06" iyz="-0.0" ixz="3e-06"/>
+  </inertial>
+  <visual>
+    <origin xyz="0.164823 0.048791 -0.341723" rpy="0 0 0"/>
     <geometry>
       <mesh filename="package://bigspot_description/meshes/RRS_1.stl" scale="0.001 0.001 0.001"/>
@@ -78,5 +158,5 @@
   </visual>
   <collision>
-    <origin xyz="-0.184517 -0.048857 -0.342398" rpy="0 0 0"/>
+    <origin xyz="0.164823 0.048791 -0.341723" rpy="0 0 0"/>
     <geometry>
       <mesh filename="package://bigspot_description/meshes/RRS_1.stl" scale="0.001 0.001 0.001"/>
@@ -84,12 +164,52 @@
   </collision>
 </link>
+<link name="RRL_1">
+  <inertial>
+    <origin xyz="0.0005644107989059011 -0.03365254077769543 -0.05152345693558058" rpy="0 0 0"/>
+    <mass value="0.25444871582041645"/>
+    <inertia ixx="0.000615" iyy="0.000574" izz="0.000105" ixy="0.0" iyz="-4e-05" ixz="4.8e-05"/>
+  </inertial>
+  <visual>
+    <origin xyz="0.133775 0.092485 -0.323" rpy="0 0 0"/>
+    <geometry>
+      <mesh filename="package://bigspot_description/meshes/RRL_1.stl" scale="0.001 0.001 0.001"/>
+    </geometry>
+    <material name="silver"/>
+  </visual>
+  <collision>
+    <origin xyz="0.133775 0.092485 -0.323" rpy="0 0 0"/>
+    <geometry>
+      <mesh filename="package://bigspot_description/meshes/RRL_1.stl" scale="0.001 0.001 0.001"/>
+    </geometry>
+  </collision>
+</link>
+<link name="RRF_1">
+  <inertial>
+    <origin xyz="-0.0015923497064600778 -0.03624611498348912 -0.0465087745386944" rpy="0 0 0"/>
+    <mass value="0.2500550328866579"/>
+    <inertia ixx="0.0007" iyy="0.000678" izz="7e-05" ixy="1e-06" iyz="2e-06" ixz="1.1e-05"/>
+  </inertial>
+  <visual>
+    <origin xyz="0.111933 0.096468 -0.181888" rpy="0 0 0"/>
+    <geometry>
+      <mesh filename="package://bigspot_description/meshes/RRF_1.stl" scale="0.001 0.001 0.001"/>
+    </geometry>
+    <material name="silver"/>
+  </visual>
+  <collision>
+    <origin xyz="0.111933 0.096468 -0.181888" rpy="0 0 0"/>
+    <geometry>
+      <mesh filename="package://bigspot_description/meshes/RRF_1.stl" scale="0.001 0.001 0.001"/>
+    </geometry>
+  </collision>
+</link>
 <link name="RLS_1">
   <inertial>
-    <origin xyz="-0.03263917034532543 -0.008846034242815902 -0.018707215426478685" rpy="0 0 0"/>
-    <mass value="0.21750157353340843"/>
-    <inertia ixx="0.000139" iyy="0.000135" izz="9.6e-05" ixy="2e-06" iyz="-0.0" ixz="-3e-06"/>
-  </inertial>
-  <visual>
-    <origin xyz="-0.184343 0.049143 -0.342368" rpy="0 0 0"/>
+    <origin xyz="0.03270821123980758 0.008996243250212595 -0.018554272527578353" rpy="0 0 0"/>
+    <mass value="0.21782970948658575"/>
+    <inertia ixx="0.000139" iyy="0.000135" izz="9.7e-05" ixy="2e-06" iyz="1e-06" ixz="3e-06"/>
+  </inertial>
+  <visual>
+    <origin xyz="0.164822 -0.049198 -0.341698" rpy="0 0 0"/>
     <geometry>
       <mesh filename="package://bigspot_description/meshes/RLS_1.stl" scale="0.001 0.001 0.001"/>
@@ -98,5 +218,5 @@
   </visual>
   <collision>
-    <origin xyz="-0.184343 0.049143 -0.342368" rpy="0 0 0"/>
+    <origin xyz="0.164822 -0.049198 -0.341698" rpy="0 0 0"/>
     <geometry>
       <mesh filename="package://bigspot_description/meshes/RLS_1.stl" scale="0.001 0.001 0.001"/>
@@ -104,12 +224,32 @@
   </collision>
 </link>
+<link name="RLL_1">
+  <inertial>
+    <origin xyz="0.0005648602121980373 0.03377765945377083 -0.051441442055425946" rpy="0 0 0"/>
+    <mass value="0.254448653712132"/>
+    <inertia ixx="0.000615" iyy="0.000574" izz="0.000105" ixy="-0.0" iyz="4.1e-05" ixz="4.8e-05"/>
+  </inertial>
+  <visual>
+    <origin xyz="0.133774 -0.092964 -0.323081" rpy="0 0 0"/>
+    <geometry>
+      <mesh filename="package://bigspot_description/meshes/RLL_1.stl" scale="0.001 0.001 0.001"/>
+    </geometry>
+    <material name="silver"/>
+  </visual>
+  <collision>
+    <origin xyz="0.133774 -0.092964 -0.323081" rpy="0 0 0"/>
+    <geometry>
+      <mesh filename="package://bigspot_description/meshes/RLL_1.stl" scale="0.001 0.001 0.001"/>
+    </geometry>
+  </collision>
+</link>
 <link name="RLF_1">
   <inertial>
-    <origin xyz="-0.0027270445134752463 -0.03603772157588159 -0.04662064942542449" rpy="0 0 0"/>
-    <mass value="0.25003083364120154"/>
-    <inertia ixx="0.000694" iyy="0.000678" izz="7.6e-05" ixy="-0.0" iyz="5e-06" ixz="-6.4e-05"/>
-  </inertial>
-  <visual>
-    <origin xyz="-0.187401 0.095965 -0.183137" rpy="0 0 0"/>
+    <origin xyz="-0.0015918551718841906 0.03635900100429153 -0.04642040795218652" rpy="0 0 0"/>
+    <mass value="0.2500551183488915"/>
+    <inertia ixx="0.0007" iyy="0.000678" izz="7e-05" ixy="-1e-06" iyz="-1e-06" ixz="1.1e-05"/>
+  </inertial>
+  <visual>
+    <origin xyz="0.111932 -0.09729 -0.181979" rpy="0 0 0"/>
     <geometry>
       <mesh filename="package://bigspot_description/meshes/RLF_1.stl" scale="0.001 0.001 0.001"/>
@@ -118,5 +258,5 @@
   </visual>
   <collision>
-    <origin xyz="-0.187401 0.095965 -0.183137" rpy="0 0 0"/>
+    <origin xyz="0.111932 -0.09729 -0.181979" rpy="0 0 0"/>
     <geometry>
       <mesh filename="package://bigspot_description/meshes/RLF_1.stl" scale="0.001 0.001 0.001"/>
@@ -124,383 +264,87 @@
   </collision>
 </link>
-<link name="RRF_1">
-  <inertial>
-    <origin xyz="-0.0022880800925702827 0.035920570914663 -0.046731066648564024" rpy="0 0 0"/>
-    <mass value="0.2500550328866579"/>
-    <inertia ixx="0.000694" iyy="0.000678" izz="7.6e-05" ixy="-0.0" iyz="-6e-06" ixz="-6.4e-05"/>
-  </inertial>
-  <visual>
-    <origin xyz="-0.187693 -0.095637 -0.182726" rpy="0 0 0"/>
-    <geometry>
-      <mesh filename="package://bigspot_description/meshes/RRF_1.stl" scale="0.001 0.001 0.001"/>
-    </geometry>
-    <material name="silver"/>
-  </visual>
-  <collision>
-    <origin xyz="-0.187693 -0.095637 -0.182726" rpy="0 0 0"/>
-    <geometry>
-      <mesh filename="package://bigspot_description/meshes/RRF_1.stl" scale="0.001 0.001 0.001"/>
-    </geometry>
-  </collision>
-</link>
-<link name="FRF_1">
-  <inertial>
-    <origin xyz="-0.0022101798151202695 0.03606539790523487 -0.04661774805926497" rpy="0 0 0"/>
-    <mass value="0.25011827063414543"/>
-    <inertia ixx="0.000694" iyy="0.000678" izz="7.6e-05" ixy="-0.0" iyz="-5e-06" ixz="-6.5e-05"/>
-  </inertial>
-  <visual>
-    <origin xyz="0.076444 -0.096255 -0.18276" rpy="0 0 0"/>
-    <geometry>
-      <mesh filename="package://bigspot_description/meshes/FRF_1.stl" scale="0.001 0.001 0.001"/>
-    </geometry>
-    <material name="silver"/>
-  </visual>
-  <collision>
-    <origin xyz="0.076444 -0.096255 -0.18276" rpy="0 0 0"/>
-    <geometry>
-      <mesh filename="package://bigspot_description/meshes/FRF_1.stl" scale="0.001 0.001 0.001"/>
-    </geometry>
-  </collision>
-</link>
-<link name="FLF_1">
-  <inertial>
-    <origin xyz="-0.002412657876597002 -0.036254756074468236 -0.04646383830667261" rpy="0 0 0"/>
-    <mass value="0.25008282200400833"/>
-    <inertia ixx="0.000694" iyy="0.000678" izz="7.6e-05" ixy="-0.0" iyz="2e-06" ixz="-6.5e-05"/>
-  </inertial>
-  <visual>
-    <origin xyz="0.077484 0.096081 -0.18294" rpy="0 0 0"/>
-    <geometry>
-      <mesh filename="package://bigspot_description/meshes/FLF_1.stl" scale="0.001 0.001 0.001"/>
-    </geometry>
-    <material name="silver"/>
-  </visual>
-  <collision>
-    <origin xyz="0.077484 0.096081 -0.18294" rpy="0 0 0"/>
-    <geometry>
-      <mesh filename="package://bigspot_description/meshes/FLF_1.stl" scale="0.001 0.001 0.001"/>
-    </geometry>
-  </collision>
-</link>
-<link name="FRL_1">
-  <inertial>
-    <origin xyz="0.013889976847389032 0.03327489929914762 -0.049659033425341115" rpy="0 0 0"/>
-    <mass value="0.2533067511311759"/>
-    <inertia ixx="0.000575" iyy="0.000567" izz="0.000135" ixy="-9e-06" iyz="3.5e-05" ixz="0.00013"/>
-  </inertial>
-  <visual>
-    <origin xyz="0.101447 -0.093082 -0.323256" rpy="0 0 0"/>
-    <geometry>
-      <mesh filename="package://bigspot_description/meshes/FRL_1.stl" scale="0.001 0.001 0.001"/>
-    </geometry>
-    <material name="silver"/>
-  </visual>
-  <collision>
-    <origin xyz="0.101447 -0.093082 -0.323256" rpy="0 0 0"/>
-    <geometry>
-      <mesh filename="package://bigspot_description/meshes/FRL_1.stl" scale="0.001 0.001 0.001"/>
-    </geometry>
-  </collision>
-</link>
-<link name="FLL_1">
-  <inertial>
-    <origin xyz="0.013702071315931347 -0.033572707159616716 -0.04951132469776853" rpy="0 0 0"/>
-    <mass value="0.2533070083934759"/>
-    <inertia ixx="0.000575" iyy="0.000566" izz="0.000136" ixy="9e-06" iyz="-3.8e-05" ixz="0.00013"/>
-  </inertial>
-  <visual>
-    <origin xyz="0.102466 0.092144 -0.323421" rpy="0 0 0"/>
-    <geometry>
-      <mesh filename="package://bigspot_description/meshes/FLL_1.stl" scale="0.001 0.001 0.001"/>
-    </geometry>
-    <material name="silver"/>
-  </visual>
-  <collision>
-    <origin xyz="0.102466 0.092144 -0.323421" rpy="0 0 0"/>
-    <geometry>
-      <mesh filename="package://bigspot_description/meshes/FLL_1.stl" scale="0.001 0.001 0.001"/>
-    </geometry>
-  </collision>
-</link>
-<link name="RLL_1">
-  <inertial>
-    <origin xyz="0.01852593549197115 -0.033435450402800715 -0.04869322173078039" rpy="0 0 0"/>
-    <mass value="0.2542264611659314"/>
-    <inertia ixx="0.000587" iyy="0.000588" izz="0.000145" ixy="1.4e-05" iyz="-3.5e-05" ixz="0.00015"/>
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