Commit message: release

File: src/bigspot_description/urdf/bigspot.xacro (robot description, xacro)
@@ -269,5 +269,5 @@
   <child link="FRS_1"/>
   <axis xyz="-0.999998 3e-05 0.001745"/>
-  <limit upper="0.523599" lower="-0.349066" effort="100" velocity="100"/>
+  <limit upper="0.523599" lower="-0.349066" effort="60.0" velocity="3"/>
 </joint>
 <joint name="FRL_Joint" type="revolute">
@@ -276,5 +276,5 @@
   <child link="FRL_1"/>
   <axis xyz="2.6e-05 0.999998 -0.002125"/>
-  <limit upper="1.570796" lower="-1.570796" effort="100" velocity="100"/>
+  <limit upper="1.570796" lower="-1.570796" effort="60.0" velocity="3"/>
 </joint>
 <joint name="FRF_Joint" type="revolute">
@@ -283,5 +283,5 @@
   <child link="FRF_1"/>
   <axis xyz="2.6e-05 0.999998 -0.002125"/>
-  <limit upper="0.0" lower="-2.617994" effort="100" velocity="100"/>
+  <limit upper="0.0" lower="-2.617994" effort="60.0" velocity="3"/>
 </joint>
 <joint name="FLS_Joint" type="revolute">
@@ -290,5 +290,5 @@
   <child link="FLS_1"/>
   <axis xyz="-0.999998 3e-05 0.001745"/>
-  <limit upper="0.349066" lower="-0.523599" effort="100" velocity="100"/>
+  <limit upper="0.349066" lower="-0.523599" effort="60.0" velocity="3"/>
 </joint>
 <joint name="FLL_Joint" type="revolute">
@@ -297,5 +297,5 @@
   <child link="FLL_1"/>
   <axis xyz="3.9e-05 0.999985 0.005513"/>
-  <limit upper="1.570796" lower="-1.570796" effort="100" velocity="100"/>
+  <limit upper="1.570796" lower="-1.570796" effort="60.0" velocity="3"/>
 </joint>
 <joint name="FLF_Joint" type="revolute">
@@ -304,5 +304,5 @@
   <child link="FLF_1"/>
   <axis xyz="-3.9e-05 -0.999985 -0.005513"/>
-  <limit upper="2.617994" lower="0.0" effort="100" velocity="100"/>
+  <limit upper="2.617994" lower="0.0" effort="60.0" velocity="3"/>
 </joint>
 <joint name="RRS_Joint" type="revolute">
@@ -311,5 +311,5 @@
   <child link="RRS_1"/>
   <axis xyz="-0.999998 7e-06 -0.001745"/>
-  <limit upper="0.523599" lower="-0.349066" effort="100" velocity="100"/>
+  <limit upper="0.523599" lower="-0.349066" effort="60.0" velocity="3"/>
 </joint>
 <joint name="RRL_Joint" type="revolute">
@@ -318,5 +318,5 @@
   <child link="RRL_1"/>
   <axis xyz="-1.5e-05 -0.999988 0.00488"/>
-  <limit upper="1.570796" lower="-1.570796" effort="100" velocity="100"/>
+  <limit upper="1.570796" lower="-1.570796" effort="60.0" velocity="3"/>
 </joint>
 <joint name="RRF_Joint" type="revolute">
@@ -325,5 +325,5 @@
   <child link="RRF_1"/>
   <axis xyz="-0.004077 0.999989 -0.002405"/>
-  <limit upper="0.0" lower="-2.792527" effort="100" velocity="100"/>
+  <limit upper="0.0" lower="-2.792527" effort="60.0" velocity="3"/>
 </joint>
 <joint name="RLS_Joint" type="revolute">
@@ -332,5 +332,5 @@
   <child link="RLS_1"/>
   <axis xyz="-0.999998 7e-06 -0.001745"/>
-  <limit upper="0.349066" lower="-0.523599" effort="100" velocity="100"/>
+  <limit upper="0.349066" lower="-0.523599" effort="60.0" velocity="3"/>
 </joint>
 <joint name="RLL_Joint" type="revolute">
@@ -339,5 +339,5 @@
   <child link="RLL_1"/>
   <axis xyz="6e-06 -0.999973 -0.007312"/>
-  <limit upper="1.570796" lower="-1.570796" effort="100" velocity="100"/>
+  <limit upper="1.570796" lower="-1.570796" effort="60.0" velocity="3"/>
 </joint>
 <joint name="RLF_Joint" type="revolute">
@@ -346,5 +346,5 @@
   <child link="RLF_1"/>
   <axis xyz="-0.004087 -0.99998 -0.004837"/>
-  <limit upper="2.792527" lower="0.0" effort="100" velocity="100"/>
+  <limit upper="2.792527" lower="0.0" effort="60.0" velocity="3"/>
 </joint>
 </robot>

Commit message: -

File: src/bigspot_description/urdf/bigspot.xacro (robot description, xacro)
@@ -269,5 +269,5 @@
   <child link="FRS_1"/>
   <axis xyz="-0.999998 3e-05 0.001745"/>
-  <limit upper="0.523599" lower="-0.349066" effort="60.0" velocity="3"/>
+  <limit upper="0.523599" lower="-0.349066" effort="15" velocity="3"/>
 </joint>
 <joint name="FRL_Joint" type="revolute">
@@ -276,5 +276,5 @@
   <child link="FRL_1"/>
   <axis xyz="2.6e-05 0.999998 -0.002125"/>
-  <limit upper="1.570796" lower="-1.570796" effort="60.0" velocity="3"/>
+  <limit upper="1.570796" lower="-1.570796" effort="15" velocity="3"/>
 </joint>
 <joint name="FRF_Joint" type="revolute">
@@ -283,5 +283,5 @@
   <child link="FRF_1"/>
   <axis xyz="2.6e-05 0.999998 -0.002125"/>
-  <limit upper="0.0" lower="-2.617994" effort="60.0" velocity="3"/>
+  <limit upper="0.0" lower="-2.617994" effort="15" velocity="3"/>
 </joint>
 <joint name="FLS_Joint" type="revolute">
@@ -290,5 +290,5 @@
   <child link="FLS_1"/>
   <axis xyz="-0.999998 3e-05 0.001745"/>
-  <limit upper="0.349066" lower="-0.523599" effort="60.0" velocity="3"/>
+  <limit upper="0.349066" lower="-0.523599" effort="15" velocity="3"/>
 </joint>
 <joint name="FLL_Joint" type="revolute">
@@ -297,5 +297,5 @@
   <child link="FLL_1"/>
   <axis xyz="3.9e-05 0.999985 0.005513"/>
-  <limit upper="1.570796" lower="-1.570796" effort="60.0" velocity="3"/>
+  <limit upper="1.570796" lower="-1.570796" effort="15" velocity="3"/>
 </joint>
 <joint name="FLF_Joint" type="revolute">
@@ -304,5 +304,5 @@
   <child link="FLF_1"/>
   <axis xyz="-3.9e-05 -0.999985 -0.005513"/>
-  <limit upper="2.617994" lower="0.0" effort="60.0" velocity="3"/>
+  <limit upper="2.617994" lower="0.0" effort="15" velocity="3"/>
 </joint>
 <joint name="RRS_Joint" type="revolute">
@@ -311,5 +311,5 @@
   <child link="RRS_1"/>
   <axis xyz="-0.999998 7e-06 -0.001745"/>
-  <limit upper="0.523599" lower="-0.349066" effort="60.0" velocity="3"/>
+  <limit upper="0.523599" lower="-0.349066" effort="15" velocity="3"/>
 </joint>
 <joint name="RRL_Joint" type="revolute">
@@ -318,5 +318,5 @@
   <child link="RRL_1"/>
   <axis xyz="-1.5e-05 -0.999988 0.00488"/>
-  <limit upper="1.570796" lower="-1.570796" effort="60.0" velocity="3"/>
+  <limit upper="1.570796" lower="-1.570796" effort="15" velocity="3"/>
 </joint>
 <joint name="RRF_Joint" type="revolute">
@@ -325,5 +325,5 @@
   <child link="RRF_1"/>
   <axis xyz="-0.004077 0.999989 -0.002405"/>
-  <limit upper="0.0" lower="-2.792527" effort="60.0" velocity="3"/>
+  <limit upper="0.0" lower="-2.792527" effort="15" velocity="3"/>
 </joint>
 <joint name="RLS_Joint" type="revolute">
@@ -332,5 +332,5 @@
   <child link="RLS_1"/>
   <axis xyz="-0.999998 7e-06 -0.001745"/>
-  <limit upper="0.349066" lower="-0.523599" effort="60.0" velocity="3"/>
+  <limit upper="0.349066" lower="-0.523599" effort="15" velocity="3"/>
 </joint>
 <joint name="RLL_Joint" type="revolute">
@@ -339,5 +339,5 @@
   <child link="RLL_1"/>
   <axis xyz="6e-06 -0.999973 -0.007312"/>
-  <limit upper="1.570796" lower="-1.570796" effort="60.0" velocity="3"/>
+  <limit upper="1.570796" lower="-1.570796" effort="15" velocity="3"/>
 </joint>
 <joint name="RLF_Joint" type="revolute">
@@ -346,5 +346,5 @@
   <child link="RLF_1"/>
   <axis xyz="-0.004087 -0.99998 -0.004837"/>
-  <limit upper="2.792527" lower="0.0" effort="60.0" velocity="3"/>
+  <limit upper="2.792527" lower="0.0" effort="15" velocity="3"/>
 </joint>
 </robot>

Commit message: -

File: src/bigspot_description/urdf/bigspot.xacro (robot description, xacro)
@@ -269,5 +269,5 @@
   <child link="FRS_1"/>
   <axis xyz="-0.999998 3e-05 0.001745"/>
-  <limit upper="0.523599" lower="-0.349066" effort="15" velocity="3"/>
+  <limit upper="0.523599" lower="-0.349066" effort="30" velocity="8"/>
 </joint>
 <joint name="FRL_Joint" type="revolute">
@@ -276,5 +276,5 @@
   <child link="FRL_1"/>
   <axis xyz="2.6e-05 0.999998 -0.002125"/>
-  <limit upper="1.570796" lower="-1.570796" effort="15" velocity="3"/>
+  <limit upper="1.570796" lower="-1.570796" effort="30" velocity="8"/>
 </joint>
 <joint name="FRF_Joint" type="revolute">
@@ -283,5 +283,5 @@
   <child link="FRF_1"/>
   <axis xyz="2.6e-05 0.999998 -0.002125"/>
-  <limit upper="0.0" lower="-2.617994" effort="15" velocity="3"/>
+  <limit upper="0.0" lower="-2.617994" effort="30" velocity="8"/>
 </joint>
 <joint name="FLS_Joint" type="revolute">
@@ -290,5 +290,5 @@
   <child link="FLS_1"/>
   <axis xyz="-0.999998 3e-05 0.001745"/>
-  <limit upper="0.349066" lower="-0.523599" effort="15" velocity="3"/>
+  <limit upper="0.349066" lower="-0.523599" effort="30" velocity="8"/>
 </joint>
 <joint name="FLL_Joint" type="revolute">
@@ -297,5 +297,5 @@
   <child link="FLL_1"/>
   <axis xyz="3.9e-05 0.999985 0.005513"/>
-  <limit upper="1.570796" lower="-1.570796" effort="15" velocity="3"/>
+  <limit upper="1.570796" lower="-1.570796" effort="30" velocity="8"/>
 </joint>
 <joint name="FLF_Joint" type="revolute">
@@ -304,5 +304,5 @@
   <child link="FLF_1"/>
   <axis xyz="-3.9e-05 -0.999985 -0.005513"/>
-  <limit upper="2.617994" lower="0.0" effort="15" velocity="3"/>
+  <limit upper="2.617994" lower="0.0" effort="30" velocity="8"/>
 </joint>
 <joint name="RRS_Joint" type="revolute">
@@ -311,5 +311,5 @@
   <child link="RRS_1"/>
   <axis xyz="-0.999998 7e-06 -0.001745"/>
-  <limit upper="0.523599" lower="-0.349066" effort="15" velocity="3"/>
+  <limit upper="0.523599" lower="-0.349066" effort="30" velocity="8"/>
 </joint>
 <joint name="RRL_Joint" type="revolute">
@@ -318,5 +318,5 @@
   <child link="RRL_1"/>
   <axis xyz="-1.5e-05 -0.999988 0.00488"/>
-  <limit upper="1.570796" lower="-1.570796" effort="15" velocity="3"/>
+  <limit upper="1.570796" lower="-1.570796" effort="30" velocity="8"/>
 </joint>
 <joint name="RRF_Joint" type="revolute">
@@ -325,5 +325,5 @@
   <child link="RRF_1"/>
   <axis xyz="-0.004077 0.999989 -0.002405"/>
-  <limit upper="0.0" lower="-2.792527" effort="15" velocity="3"/>
+  <limit upper="0.0" lower="-2.792527" effort="30" velocity="8"/>
 </joint>
 <joint name="RLS_Joint" type="revolute">
@@ -332,5 +332,5 @@
   <child link="RLS_1"/>
   <axis xyz="-0.999998 7e-06 -0.001745"/>
-  <limit upper="0.349066" lower="-0.523599" effort="15" velocity="3"/>
+  <limit upper="0.349066" lower="-0.523599" effort="30" velocity="8"/>
 </joint>
 <joint name="RLL_Joint" type="revolute">
@@ -339,5 +339,5 @@
   <child link="RLL_1"/>
   <axis xyz="6e-06 -0.999973 -0.007312"/>
-  <limit upper="1.570796" lower="-1.570796" effort="15" velocity="3"/>
+  <limit upper="1.570796" lower="-1.570796" effort="30" velocity="8"/>
 </joint>
 <joint name="RLF_Joint" type="revolute">
@@ -346,5 +346,5 @@
   <child link="RLF_1"/>
   <axis xyz="-0.004087 -0.99998 -0.004837"/>
-  <limit upper="2.792527" lower="0.0" effort="15" velocity="3"/>
+  <limit upper="2.792527" lower="0.0" effort="30" velocity="8"/>
 </joint>
 </robot>

Commit message: add world

File: src/bigspot_description/urdf/bigspot.xacro (robot description, xacro)
@@ -24,4 +24,36 @@
   </collision>
 </link>
+<link name='camera_link'>
+  <pose frame=''>0.1 0 0 0 0 0</pose>
+  <inertial>
+    <pose frame=''>0.01 0.025 0.025 0 -0 0</pose>
+    <mass>0.01</mass>
+    <inertia>
+      <ixx>4.15e-06</ixx>
+      <ixy>0</ixy>
+      <ixz>0</ixz>
+      <iyy>2.407e-06</iyy>
+      <iyz>0</iyz>
+      <izz>2.407e-06</izz>
+    </inertia>
+  </inertial>
+  <self_collide>0</self_collide>
+  <kinematic>0</kinematic>
+  <visual name='visual'>
+    <geometry>
+      <box>
+        <size>0.026012 0.029339 0.024291</size>
+      </box>
+    </geometry>
+    <pose frame=''>0 0 0 0 -0 0</pose>
+    <cast_shadows>1</cast_shadows>
+    <transparency>0</transparency>
+  </visual>
+</link>
+<joint name="camera_joint" type="fixed">
+  <origin xyz="0.021842 -0.003983 -0.141112" rpy="0 0 0"/>
+  <parent link="base_link"/>
+  <child link="camera_link"/>
+</joint>
 <link name="FRS_1">
   <inertial>

Commit message: add  camera

File: src/bigspot_description/urdf/bigspot.xacro (robot description, xacro)
@@ -4,4 +4,5 @@
 <xacro:include filename="$(find bigspot_description)/urdf/bigspot.trans" />
 <xacro:include filename="$(find bigspot_description)/urdf/bigspot.gazebo" />
+<xacro:property name="camera_link" value="0.05" /> <!-- Size of square 'camera' box -->
 <link name="base_link">
   <inertial>
@@ -24,36 +25,31 @@
   </collision>
 </link>
-<link name='camera_link'>
-  <pose frame=''>0.1 0 0 0 0 0</pose>
-  <inertial>
-    <pose frame=''>0.01 0.025 0.025 0 -0 0</pose>
-    <mass>0.01</mass>
-    <inertia>
-      <ixx>4.15e-06</ixx>
-      <ixy>0</ixy>
-      <ixz>0</ixz>
-      <iyy>2.407e-06</iyy>
-      <iyz>0</iyz>
-      <izz>2.407e-06</izz>
-    </inertia>
-  </inertial>
-  <self_collide>0</self_collide>
-  <kinematic>0</kinematic>
-  <visual name='visual'>
-    <geometry>
-      <box>
-        <size>0.026012 0.029339 0.024291</size>
-      </box>
-    </geometry>
-    <pose frame=''>0 0 0 0 -0 0</pose>
-    <cast_shadows>1</cast_shadows>
-    <transparency>0</transparency>
-  </visual>
-</link>
-<joint name="camera_joint" type="fixed">
-  <origin xyz="0.021842 -0.003983 -0.141112" rpy="0 0 0"/>
-  <parent link="base_link"/>
-  <child link="camera_link"/>
-</joint>
+  <joint name="camera_joint" type="fixed">
+    <axis xyz="0 1 0" />
+    <origin xyz="${camera_link} 0 0" rpy="0 0 0"/>
+    <parent link="base_link"/>
+    <child link="camera_link"/>
+  </joint>
+  <!-- Camera -->
+  <link name="camera_link">
+    <collision>
+      <origin xyz="0 0 0" rpy="0 0 0"/>
+      <geometry>
+    <box size="${camera_link} ${camera_link} ${camera_link}"/>
+      </geometry>
+    </collision>
+    <visual>
+      <origin xyz="0 0 0" rpy="0 0 0"/>
+      <geometry>
+    <box size="${camera_link} ${camera_link} ${camera_link}"/>
+      </geometry>
+      <material name="red"/>
+    </visual>
+    <inertial>
+      <mass value="1e-5" />
+      <origin xyz="0 0 0" rpy="0 0 0"/>
+      <inertia ixx="1e-6" ixy="0" ixz="0" iyy="1e-6" iyz="0" izz="1e-6" />
+    </inertial>
+  </link>
 <link name="FRS_1">
   <inertial>

File: src/bigspot_description/urdf/materials.xacro (robot description, xacro)
@@ -4,3 +4,24 @@
   <color rgba="0.700 0.700 0.700 1.000"/>
 </material>
+<material name="blue">
+  <color rgba="0.0 0.0 0.8 1.0"/>
+</material>
+<material name="green">
+  <color rgba="0.0 0.8 0.0 1.0"/>
+</material>
+<material name="gray">
+  <color rgba="0.7 0.7 0.7 1.0"/>
+</material>
+<material name="darkgray">
+  <color rgba="0.3 0.3 0.3 1.0"/>
+</material>
+<material name="red">
+  <color rgba="0.8 0.0 0.0 1.0"/>
+</material>
+<material name="white">
+  <color rgba="1.0 1.0 1.0 1.0"/>
+</material>
+<material name="yellow">
+  <color rgba="0.8 0.8 0.0 1.0"/>
+</material>
 </robot>

Commit message: add sonar

File: src/bigspot_description/urdf/bigspot.xacro (robot description, xacro)
@@ -53,4 +53,29 @@
   </link>
 -->
+<joint name="ir_front_joint" type="fixed">
+    <axis xyz="0 1 0" />
+    <origin rpy="0 0 0" xyz="0.18 0 0.35" />
+    <parent link="base_link"/>
+    <child link="base_ir_front"/>
+</joint>
+<link name="base_ir_front">
+    <collision>
+      <origin xyz="0 0 0" rpy="0 0 0"/>
+      <geometry>
+        <box size="0.01 0.01 0.01"/>
+      </geometry>
+    </collision>
+    <visual>
+      <origin xyz="0 0 0" rpy="0 0 0"/>
+      <geometry>
+        <box size="0.01 0.01 0.01"/>
+      </geometry>
+    </visual>
+    <inertial>
+      <mass value="1e-5" />
+      <origin xyz="0 0 0" rpy="0 0 0"/>
+      <inertia ixx="1e-6" ixy="0" ixz="0" iyy="1e-6" iyz="0"      izz="1e-6" />
+    </inertial>
+</link>
 <link name="FRS_1">
   <inertial>
