Commit message: Refine Pi4 R2 CAD and validate recorded motion with video gallery

File: design/pi4/bigspot.urdf (robot description, URDF)
Before this commit: robot bigspot_autonomy, 15 links, 14 joints
Links:
- link FL_abduction_link: mass 0.4781603552900706 -> 0.49530215589264903
- link FL_lower_link: mass 0.12406838068242512 -> 0.14694892944839885; geometry collision box size=0.018 0.012 0.014; collision box size=0.025 0.04 0.007
- link FL_upper_link: mass 0.5020334705223707 -> 0.49855400195496596; geometry collision box size=0.026 0.012 0.1; collision cylinder length=0.0455 radius=0.03925
- link FR_abduction_link: mass 0.4781603552900706 -> 0.4953021558912428
- link FR_lower_link: mass 0.12406838068242512 -> 0.14694892944839882; geometry collision box size=0.018 0.012 0.014; collision box size=0.025 0.04 0.007
- link FR_upper_link: mass 0.5020334705223707 -> 0.4985540019549658; geometry collision box size=0.026 0.012 0.1; collision cylinder length=0.0455 radius=0.03925
- link RL_abduction_link: mass 0.4781603552900706 -> 0.4953021558911146
- link RL_lower_link: mass 0.12406838068242512 -> 0.14694892944839885; geometry collision box size=0.018 0.012 0.014; collision box size=0.025 0.04 0.007
- link RL_upper_link: mass 0.5020334705223707 -> 0.49855400195496596; geometry collision box size=0.026 0.012 0.1; collision cylinder length=0.0455 radius=0.03925
- link RR_abduction_link: mass 0.4781603552900706 -> 0.4953021558875289
- link RR_lower_link: mass 0.12406838068242512 -> 0.14694892944839882; geometry collision box size=0.018 0.012 0.014; collision box size=0.025 0.04 0.007
- link RR_upper_link: mass 0.5020334705223707 -> 0.4985540019549658; geometry collision box size=0.026 0.012 0.1; collision cylinder length=0.0455 radius=0.03925
- link base_link: mass 4.796673432111005 -> 4.90479585814143; geometry collision box size=0.003 0.018 0.084; collision box size=0.003 0.018 0.084
Joints:
- joint FL_knee: limit lower=0.1 upper=3.0 effort=17.0 velocity=12 -> lower=0.1 upper=2.55 effort=17.0 velocity=12
- joint FR_knee: limit lower=0.1 upper=3.0 effort=17.0 velocity=12 -> lower=0.1 upper=2.55 effort=17.0 velocity=12
- joint RL_knee: limit lower=0.1 upper=3.0 effort=17.0 velocity=12 -> lower=0.1 upper=2.55 effort=17.0 velocity=12
- joint RR_knee: limit lower=0.1 upper=3.0 effort=17.0 velocity=12 -> lower=0.1 upper=2.55 effort=17.0 velocity=12

Commit message: Add SPORT CAD, complete motion regeneration and reliable ranged video playback

File: design/pi4/bigspot.urdf (robot description, URDF)
Before this commit: robot bigspot_autonomy, 15 links, 14 joints
Links:
- link FL_abduction_link: mass 0.49530215589264903 -> 0.5065781470343673; geometry collision cylinder length=0.002 radius=0.0395; collision cylinder length=0.0455 radius=0.03925
- link FL_lower_link: geometry collision box size=0.018 0.012 0.014; collision box size=0.025 0.04 0.007
- link FL_upper_link: mass 0.49855400195496596 -> 0.5098299930966843; geometry collision box size=0.026 0.012 0.1; collision cylinder length=0.002 radius=0.0395
- link FR_abduction_link: mass 0.4953021558912428 -> 0.5065781470329611; geometry collision cylinder length=0.002 radius=0.0395; collision cylinder length=0.0455 radius=0.03925
- link FR_lower_link: geometry collision box size=0.018 0.012 0.014; collision box size=0.025 0.04 0.007
- link FR_upper_link: mass 0.4985540019549658 -> 0.5098299930966841; geometry collision box size=0.026 0.012 0.1; collision cylinder length=0.002 radius=0.0395
- link RL_abduction_link: mass 0.4953021558911146 -> 0.5065781470328329; geometry collision cylinder length=0.002 radius=0.0395; collision cylinder length=0.0455 radius=0.03925
- link RL_lower_link: geometry collision box size=0.018 0.012 0.014; collision box size=0.025 0.04 0.007
- link RL_upper_link: mass 0.49855400195496596 -> 0.5098299930966843; geometry collision box size=0.026 0.012 0.1; collision cylinder length=0.002 radius=0.0395
- link RR_abduction_link: mass 0.4953021558875289 -> 0.5065781470292472; geometry collision cylinder length=0.002 radius=0.0395; collision cylinder length=0.0455 radius=0.03925
- link RR_lower_link: geometry collision box size=0.018 0.012 0.014; collision box size=0.025 0.04 0.007
- link RR_upper_link: mass 0.4985540019549658 -> 0.5098299930966841; geometry collision box size=0.026 0.012 0.1; collision cylinder length=0.002 radius=0.0395
- link base_link: mass 4.90479585814143 -> 5.180523313622426; geometry collision box size=0.002 0.118 0.056; collision box size=0.002 0.118 0.056
Joints:
- joint camera_link_mount: origin xyz=0.205 0 0.075 rpy=0 0.20943951 0 -> xyz=0.205 0 0.07 rpy=0 0.20943951 0
